Commit message: sdf, urdf and folder modifications

File: src/ur5_softmat/models/universal-robot-ur5/ur5robot.urdf (robot description, URDF)
Before this commit: robot universal-robot-ur5, 9 links, 8 joints
Links:
- link base_link: geometry collision mesh filename=package://./meshes/ur5/collision/Base.dae; visual mesh filename=package://./meshes/ur5/visual/Base.dae
- link forearm_link: geometry collision mesh filename=package://./meshes/ur5/collision/Forearm.dae; visual mesh filename=package://./meshes/ur5/visual/Forearm.dae
- link shoulder_link: geometry collision mesh filename=package://./meshes/ur5/collision/Shoulder.dae; visual mesh filename=package://./meshes/ur5/visual/Shoulder.dae
- link upper_arm_link: geometry collision mesh filename=package://./meshes/ur5/collision/UpperArm.dae; visual mesh filename=package://./meshes/ur5/visual/UpperArm.dae
- link wrist_1_link: geometry collision mesh filename=package://./meshes/ur5/collision/Wrist1.dae; visual mesh filename=package://./meshes/ur5/visual/Wrist1.dae
- link wrist_2_link: geometry collision mesh filename=package://./meshes/ur5/collision/Wrist2.dae; visual mesh filename=package://./meshes/ur5/visual/Wrist2.dae
- link wrist_3_link: geometry collision mesh filename=package://./meshes/ur5/collision/Wrist3.dae; visual mesh filename=package://./meshes/ur5/visual/Wrist3.dae

File: src/ur5_softmat/models/universal-robot-ur5/ur5robot_old.urdf (robot description, URDF)
Before this commit: robot universal-robot-ur5, 9 links, 8 joints
Links:
- link base_link: geometry collision mesh filename=package://./meshes/ur5/collision/Base.dae; visual mesh filename=package://./meshes/ur5/visual/Base.dae
- link ee_link: mass 0.00001 -> None; geometry 
- link forearm_link: geometry collision mesh filename=package://./meshes/ur5/collision/Forearm.dae; visual mesh filename=package://./meshes/ur5/visual/Forearm.dae
- link shoulder_link: geometry collision mesh filename=package://./meshes/ur5/collision/Shoulder.dae; visual mesh filename=package://./meshes/ur5/visual/Shoulder.dae
- link upper_arm_link: geometry collision mesh filename=package://./meshes/ur5/collision/UpperArm.dae; visual mesh filename=package://./meshes/ur5/visual/UpperArm.dae
- link wrist_1_link: geometry collision mesh filename=package://./meshes/ur5/collision/Wrist1.dae; visual mesh filename=package://./meshes/ur5/visual/Wrist1.dae
- link wrist_2_link: geometry collision mesh filename=package://./meshes/ur5/collision/Wrist2.dae; visual mesh filename=package://./meshes/ur5/visual/Wrist2.dae
- link wrist_3_link: geometry collision mesh filename=package://./meshes/ur5/collision/Wrist3.dae; visual mesh filename=package://./meshes/ur5/visual/Wrist3.dae
Joints:
- removed joint world_base_joint
- added joint fixed: type fixed, parent world, child base_link
- joint ee_fixed_joint: axis 0 1 0 -> (none); limit lower=0 upper=0 effort=0.0 velocity=0 -> (none); type revolute -> fixed
- joint wrist_1_joint: limit lower=-3.14159265 upper=4.71 effort=28.0 velocity=3.14159265 -> lower=-3.14159265 upper=0.7853981625 effort=28.0 velocity=3.14159265
- joint wrist_2_joint: limit lower=-3.14159265 upper=4.71 effort=28.0 velocity=3.14159265 -> lower=-3.14159265 upper=3.14159265 effort=28.0 velocity=3.14159265
