Commit message: editing sdf and urdf files

File: src/ur5_softmat/urdf/ur5e.urdf (robot description, URDF)
Before this commit: robot universal-robot-ur5, 9 links, 8 joints
Links:
- link base_link: geometry collision mesh filename=package://ur5_softmat/models/ur5e/meshes/collision/Base.dae; visual mesh filename=package://ur5_softmat/models/ur5e/meshes/visual/Base.dae
- link forearm_link: geometry collision mesh filename=package://ur5_softmat/models/ur5e/meshes/collision/Forearm.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; visual mesh filename=package://ur5_softmat/models/ur5e/meshes/visual/Forearm.dae
- link shoulder_link: geometry collision mesh filename=package://ur5_softmat/models/ur5e/meshes/collision/Shoulder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; visual mesh filename=package://ur5_softmat/models/ur5e/meshes/visual/Shoulder.dae
- link upper_arm_link: geometry collision mesh filename=package://ur5_softmat/models/ur5e/meshes/collision/UpperArm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; visual mesh filename=package://ur5_softmat/models/ur5e/meshes/visual/UpperArm.dae
- link wrist_1_link: geometry collision mesh filename=package://ur5_softmat/models/ur5e/meshes/collision/Wrist1.d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; visual mesh filename=package://ur5_softmat/models/ur5e/meshes/visual/Wrist1.dae
- link wrist_2_link: geometry collision mesh filename=package://ur5_softmat/models/ur5e/meshes/collision/Wrist2.d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; visual mesh filename=package://ur5_softmat/models/ur5e/meshes/visual/Wrist2.dae
- link wrist_3_link: geometry collision mesh filename=package://ur5_softmat/models/ur5e/meshes/collision/Wrist3.d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; visual mesh filename=package://ur5_softmat/models/ur5e/meshes/visual/Wrist3.dae

Commit message: sdf edits

File: src/ur5_softmat/urdf/ur5e.urdf (robot description, URDF)
Before this commit: robot universal-robot-ur5, 9 links, 8 joints
Links:
- link base_link: geometry collision mesh filename=package://ur5_softmat/models/ur5e/meshes/collision/base.stl scale=1.0 1.0 1.0; visual mesh filename=package://ur5_softmat/models/ur5e/meshes/visual/base.dae
- link forearm_link: geometry collision mesh filename=package://ur5_softmat/models/ur5e/meshes/collision/forearm.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 scale=1.0 1.0 1.0; visual mesh filename=package://ur5_softmat/models/ur5e/meshes/visual/forearm.dae
- link shoulder_link: geometry collision mesh filename=package://ur5_softmat/models/ur5e/meshes/collision/shoulder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 scale=1.0 1.0 1.0; visual mesh filename=package://ur5_softmat/models/ur5e/meshes/visual/shoulder.dae
- link upper_arm_link: geometry collision mesh filename=package://ur5_softmat/models/ur5e/meshes/collision/upperarm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 scale=1.0 1.0 1.0; visual mesh filename=package://ur5_softmat/models/ur5e/meshes/visual/upperarm.dae
- link wrist_1_link: geometry collision mesh filename=package://ur5_softmat/models/ur5e/meshes/collision/wrist1.s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 scale=1.0 1.0 1.0; visual mesh filename=package://ur5_softmat/models/ur5e/meshes/visual/wrist1.dae
- link wrist_2_link: geometry collision mesh filename=package://ur5_softmat/models/ur5e/meshes/collision/wrist2.s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 scale=1.0 1.0 1.0; visual mesh filename=package://ur5_softmat/models/ur5e/meshes/visual/wrist2.dae
- link wrist_3_link: geometry collision mesh filename=package://ur5_softmat/models/ur5e/meshes/collision/wrist3.s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 scale=1.0 1.0 1.0; visual mesh filename=package://ur5_softmat/models/ur5e/meshes/visual/wrist3.dae
